File: tracking_device.sch (KiCad schematic (older format))
At the start: 50 parts, among them J1 USB_OTG, J2 CONN_COAXIAL, J3 JST-PH, J4 Micro_SD_Card, Q1 PMGD280UN, U1 RClamp0503F, U2 LDK220M30R, U3 MCP73831, U4 MAX-M8, U5 STC3100

Commit message: Most components arranged on PCB
Parts:
- removed J4: Micro_SD_Card, symbol Micro_SD_Card
- added J4: Micro_SD_Connector, tracking_device:SD_Card_Connector_Ebay, symbol Micro_SD_Connector
- C1, C10, C12, C4: footprint (none) -> Capacitors_SMD:C_0805_HandSoldering
- D1: footprint footprints:DO-214AC -> tracking_device:DO-214AC
- J1: footprint footprints:FCI_10118192-0001LF -> tracking_device:FCI_10118192-0001LF
- J2: footprint (none) -> tracking_device:RP-SMA
- J3: footprint (none) -> Connectors_JST:JST_PH_S2B-PH-SM4-TB_02x2.00mm_Angled
- L1: footprint (none) -> Inductors_SMD:L_0805_HandSoldering
- MK1: footprint footprints:MIC_3x4 -> tracking_device:MIC_3x4
- Q1: footprint footprints:SOT-363_SC-70-6_Handsoldering -> tracking_device:SOT-363_SC-70-6_Handsoldering
- R23: footprint (none) -> Resistors_SMD:R_0805_HandSoldering
- U1: footprint footprints:SOT-353_SC-70-5_Handsoldering -> tracking_device:SOT-353_SC-70-5_Handsoldering
- U2: footprint footprints:SOT-23-5_HandSoldering -> tracking_device:SOT-23-5_HandSoldering
- U4: footprint manuf:U-BLOX_MAX -> tracking_device:U-BLOX_MAX-M8
- gave numbers to parts that had none: 5
Connections:
- net labels added: GPS_ANT, SD_CK, SD_CMD, SD_D0, SD_D1, SD_D2, SD_D3, USB_D+, USB_D-
- net labels removed: USB_DM, USB_DP
- wire segments 201 -> 208
Other:
- note added: "which pin is +??"

Commit message: Version sent out for fabrication
Parts:
- added J3, J4, J5, J6: CONN_01X02, tracking_device:Pin_Header_Straight_2x01_Pitch2.54mm, symbol CONN_01X02
- added MH1, MH2, MH3: MOUNTING_HOLE, Mounting_Holes:MountingHole_2.2mm_M2, symbol MOUNTING_HOLE
- added R4: 10k, Resistors_SMD:R_0805_HandSoldering, symbol R
- added R5: 5.6k, Resistors_SMD:R_0805_HandSoldering, symbol R
- added SW1, SW2: SW_SPDT, tracking_device:CSS-1210TB, symbol SW_SPDT
- added TP1, TP10, TP11, TP2, TP3, TP4, TP5, TP6, TP7, TP8, TP9: TEST, Measurement_Points:Measurement_Point_Round-TH_Small, symbol TEST
- J7: renamed from J3; footprint Connectors_JST:JST_PH_S2B-PH-SM4-TB_02x2.00mm_Angled -> tracking_device:JST_PH_S2B-PH-SM4-TB_02x2.00mm_Angled
- R12: renamed from R5; value 100 -> 100 (DNI)
- R14: renamed from R6; value 10k -> 10k (DNI)
- R15: renamed from R12; value 12 -> DNI
- R16: renamed from R14; value 500k -> 12k
- U5: footprint Housings_SSOP:MSOP-8_3x3mm_Pitch0.65mm -> Housings_DFN_QFN:DFN-8-1EP_3x3mm_Pitch0.5mm
- renumbered C11 to C10, C10 to C11, J4 to J8, R3 to R1, R15 to R17, R16 to R18, R17 to R19, R1 to R2, R18 to R20, R19 to R21, R20 to R22, R21 to R23, R22 to R24, R23 to R25, R2 to R3, R4 to R6, U4 to U3, U3 to U4
Connections:
- net GND: now also C1.1, Q1.1 (S), MH1.~, MH2.~, MH3.~, R5.1, SW1.3 (C), SW2.3 (C); no longer C1.2, R15.1
- net GPS_EXTINT: now also TP3.1; no longer U3.4 (TIMEPULSE)
- net GPS_I2C_SCL: now also J3.1 (P1)
- net GPS_I2C_SDA: now also J3.2 (P2)
- net GPS_RESET_N: now also TP4.1
- net GPS_UART_RX: now also J4.1 (P1)
- net GPS_UART_TX: now also J4.2 (P2)
- net LSE_CLK: now also TP9.1
- net MIC_CLK: now also TP7.1
- net MIC_DATA: now also TP8.1
- net PMIC_FAST: now also TP11.1
- net PMIC_I2C_SCL: now also J5.1 (P1)
- net PMIC_I2C_SDA: now also J5.2 (P2)
- net PMIC_STAT: now also TP10.1
- net VBAT: now also C1.2, J6.1 (P1); no longer C1.1
- net VDD: now also R4.2, SW1.1 (A), SW2.1 (A)
- net VUSB: now also TP1.1
- net VUSB_DET: now also TP2.1
- net at J7.2 (P2), R25.1, U5.6 (CG): now also J6.2 (P2)
- net at R16.1, U4.5 (PROG): now also R15.2, TP6.1; no longer Q1.3 (D)
- net at U2.4 (ADJ): now also R4.1, R5.2
- new net: Q1.3 (D), R15.1
- new net GPS_TIMEPULSE: TP5.1, U3.4 (TIMEPULSE)
- new net Microcontroller/SWITCH_1: SW1.2 (B)
- new net Microcontroller/SWITCH_2: SW2.2 (B)
- no-connect marks 7 -> 5
Other:
- moved on the sheet: C1, C11, C12, C2, C4, C6, C7, C8, J2, J8, L1, MK1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

Commit message: Rev 1 sent for fabrication
Parts:
- R12: value 100 (DNI) -> 100
- R14: value 10k (DNI) -> 10k
- R15: value DNI -> 4k
- R4: value 10k -> 12k
- R5: value 5.6k -> 20k
Other:
- moved on the sheet: MH1, MH2, MH3, Q1B, TP10, TP2, TP3, TP4, TP5, TP8, TP9
Changed lines of the file:
@@
 encoding utf-8
 Sheet 1 3
-Title "Tracking Device"
-Date "2017-08-08"
+Title "Spy Thing"
+Date "2017-07-08"
 Rev "1"
 Comp ""
@@
 P 4400 1450
 F 0 "R15" V 4480 1450 50  0000 C CNN
-F 1 "DNI" V 4400 1450 50  0000 C CNN
+F 1 "4k" V 4400 1450 50  0000 C CNN
 F 2 "Resistors_SMD:R_0805_HandSoldering" V 4330 1450 50  0001 C CNN
 F 3 "" H 4400 1450 50  0001 C CNN
@@
 L PMGD280UN Q1
 U 2 1 59B0AEBF
-P 5700 2400
-F 0 "Q1" H 5900 2450 50  0000 L CNN
-F 1 "PMGD280UN" H 5900 2350 50  0000 L CNN
-F 2 "" H 5900 2500 50  0001 C CNN
-F 3 "" H 5700 2400 50  0001 C CNN
-	2    5700 2400
+P 5500 2200
+F 0 "Q1" H 5700 2250 50  0000 L CNN
+F 1 "PMGD280UN" H 5700 2150 50  0000 L CNN
+F 2 "" H 5700 2300 50  0001 C CNN
+F 3 "" H 5500 2200 50  0001 C CNN
+	2    5500 2200
 	1    0    0    -1
 $EndComp
@@
 P 4150 1300
 F 0 "R14" V 4230 1300 50  0000 C CNN
-F 1 "10k (DNI)" V 4150 1300 50  0000 C CNN
+F 1 "10k" V 4150 1300 50  0000 C CNN
 F 2 "Resistors_SMD:R_0805_HandSoldering" V 4080 1300 50  0001 C CNN
 F 3 "" H 4150 1300 50  0001 C CNN
@@
 P 3900 2000
 F 0 "R12" V 3980 2000 50  0000 C CNN
-F 1 "100 (DNI)" V 3900 2000 50  0000 C CNN
+F 1 "100" V 3900 2000 50  0000 C CNN
 F 2 "Resistors_SMD:R_0805_HandSoldering" V 3830 2000 50  0001 C CNN
 F 3 "" H 3900 2000 50  0001 C CNN
@@
 	1    0    0    -1
 $EndComp
-Text Notes 550  5650 0    60   ~ 0
+Text Notes 500  5750 0    60   ~ 0
 VCC_RF is for powering active\nantenna if it also operates at VCC\nDNI inductor if not used
 $Comp
@@
 	1    0    0    -1
 $EndComp
-Text Notes 3450 8000 0    60   ~ 0
+Text Notes 3350 7950 0    60   ~ 0
 Default 0x42 I2C address
 NoConn ~ 3050 6550
@@
 Text Label 7650 5200 2    60   ~ 0
 PMIC_FAST
-NoConn ~ 5800 2200
-NoConn ~ 5500 2400
-NoConn ~ 5800 2600
+NoConn ~ 5600 2000
+NoConn ~ 5300 2200
+NoConn ~ 5600 2400
 $Comp
 L R R19
@@
 L MOUNTING_HOLE MH1
 U 1 1 59FBDF84
-P 5600 6900
-F 0 "MH1" H 5600 7000 40  0000 C CNN
-F 1 "MOUNTING_HOLE" H 5600 6800 40  0000 C CNN
-F 2 "Mounting_Holes:MountingHole_2.2mm_M2" H 5600 6900 60  0000 C CNN
-F 3 "" H 5600 6900 60  0000 C CNN
-	1    5600 6900
+P 5200 6850
+F 0 "MH1" H 5200 6950 40  0000 C CNN
+F 1 "MOUNTING_HOLE" H 5200 6750 40  0000 C CNN
+F 2 "Mounting_Holes:MountingHole_2.2mm_M2" H 5200 6850 60  0001 C CNN
+F 3 "" H 5200 6850 60  0000 C CNN
+	1    5200 6850
 	1    0    0    -1
 $EndComp
@@
 L GND #PWR043
 U 1 1 59FC06A9
-P 5250 7700
-F 0 "#PWR043" H 5250 7450 50  0001 C CNN
-F 1 "GND" H 5250 7550 50  0000 C CNN
-F 2 "" H 5250 7700 50  0001 C CNN
-F 3 "" H 5250 7700 50  0001 C CNN
-	1    5250 7700
+P 4850 7650
+F 0 "#PWR043" H 4850 7400 50  0001 C CNN
+F 1 "GND" H 4850 7500 50  0000 C CNN
+F 2 "" H 4850 7650 50  0001 C CNN
+F 3 "" H 4850 7650 50  0001 C CNN
+	1    4850 7650
 	-1   0    0    -1
 $EndComp
@@
 L MOUNTING_HOLE MH2
 U 1 1 59FBEE8D
-P 5600 7200
-F 0 "MH2" H 5600 7300 40  0000 C CNN
-F 1 "MOUNTING_HOLE" H 5600 7100 40  0000 C CNN
-F 2 "Mounting_Holes:MountingHole_2.2mm_M2" H 5600 7200 60  0000 C CNN
-F 3 "" H 5600 7200 60  0000 C CNN
-	1    5600 7200
+P 5200 7150
+F 0 "MH2" H 5200 7250 40  0000 C CNN
+F 1 "MOUNTING_HOLE" H 5200 7050 40  0000 C CNN
+F 2 "Mounting_Holes:MountingHole_2.2mm_M2" H 5200 7150 60  0001 C CNN
+F 3 "" H 5200 7150 60  0000 C CNN
+	1    5200 7150
 	1    0    0    -1
 $EndComp
@@
 L MOUNTING_HOLE MH3
 U 1 1 59FBF08E
-P 5600 7500
-F 0 "MH3" H 5600 7600 40  0000 C CNN
-F 1 "MOUNTING_HOLE" H 5600 7400 40  0000 C CNN
-F 2 "Mounting_Holes:MountingHole_2.2mm_M2" H 5600 7500 60  0000 C CNN
-F 3 "" H 5600 7500 60  0000 C CNN
-	1    5600 7500
+P 5200 7450
+F 0 "MH3" H 5200 7550 40  0000 C CNN
+F 1 "MOUNTING_HOLE" H 5200 7350 40  0000 C CNN
+F 2 "Mounting_Holes:MountingHole_2.2mm_M2" H 5200 7450 60  0001 C CNN
+F 3 "" H 5200 7450 60  0000 C CNN
+	1    5200 7450
 	1    0    0    -1
 $EndComp
@@
 F 3 "" H 3600 5350 50  0001 C CNN
 	1    3600 5350
-	0    -1   -1   0
+	1    0    0    -1
 $EndComp
 $Comp
 L TEST TP3
 U 1 1 59FCDF58
-P 3600 5450
-F 0 "TP3" H 3600 5750 50  0000 C BNN
-F 1 "TEST" H 3600 5700 50  0000 C CNN
-F 2 "Measurement_Points:Measurement_Point_Round-TH_Small" H 3600 5450 50  0001 C CNN
-F 3 "" H 3600 5450 50  0001 C CNN
-	1    3600 5450
-	0    -1   -1   0
+P 3450 5450
+F 0 "TP3" H 3450 5750 50  0000 C BNN
+F 1 "TEST" H 3450 5700 50  0000 C CNN
+F 2 "Measurement_Points:Measurement_Point_Round-TH_Small" H 3450 5450 50  0001 C CNN
+F 3 "" H 3450 5450 50  0001 C CNN
+	1    3450 5450
+	1    0    0    -1
 $EndComp
 $Comp
 L TEST TP4
 U 1 1 59FCE164
-P 3600 5550
-F 0 "TP4" H 3600 5850 50  0000 C BNN
-F 1 "TEST" H 3600 5800 50  0000 C CNN
-F 2 "Measurement_Points:Measurement_Point_Round-TH_Small" H 3600 5550 50  0001 C CNN
-F 3 "" H 3600 5550 50  0001 C CNN
-	1    3600 5550
-	0    -1   -1   0
+P 3250 5500
+F 0 "TP4" H 3250 5800 50  0000 C BNN
+F 1 "TEST" H 3250 5750 50  0000 C CNN
+F 2 "Measurement_Points:Measurement_Point_Round-TH_Small" H 3250 5500 50  0001 C CNN
+F 3 "" H 3250 5500 50  0001 C CNN
+	1    3250 5500
+	1    0    0    -1
 $EndComp
 $Comp
 L TEST TP5
 U 1 1 59FCE373
-P 3600 5650
-F 0 "TP5" H 3600 5950 50  0000 C BNN
-F 1 "TEST" H 3600 5900 50  0000 C CNN
-F 2 "Measurement_Points:Measurement_Point_Round-TH_Small" H 3600 5650 50  0001 C CNN
-F 3 "" H 3600 5650 50  0001 C CNN
-	1    3600 5650
-	0    -1   -1   0
+P 3050 5500
+F 0 "TP5" H 3050 5800 50  0000 C BNN
+F 1 "TEST" H 3050 5750 50  0000 C CNN
+F 2 "Measurement_Points:Measurement_Point_Round-TH_Small" H 3050 5500 50  0001 C CNN
+F 3 "" H 3050 5500 50  0001 C CNN
+	1    3050 5500
+	1    0    0    -1
 $EndComp
 $Comp
@@
 L TEST TP10
 U 1 1 59FCF3DE
-P 7650 5100
-F 0 "TP10" H 7650 5400 50  0000 C BNN
-F 1 "TEST" H 7650 5350 50  0000 C CNN
-F 2 "Measurement_Points:Measurement_Point_Round-TH_Small" H 7650 5100 50  0001 C CNN
-F 3 "" H 7650 5100 50  0001 C CNN
-	1    7650 5100
+P 7650 5000
+F 0 "TP10" H 7650 5300 50  0000 C BNN
+F 1 "TEST" H 7650 5250 50  0000 C CNN
+F 2 "Measurement_Points:Measurement_Point_Round-TH_Small" H 7650 5000 50  0001 C CNN
+F 3 "" H 7650 5000 50  0001 C CNN
+	1    7650 5000
 	0    1    1    0
 $EndComp
@@
 L TEST TP8
 U 1 1 59FD0A58
-P 7650 4150
-F 0 "TP8" H 7650 4450 50  0000 C BNN
-F 1 "TEST" H 7650 4400 50  0000 C CNN
-F 2 "Measurement_Points:Measurement_Point_Round-TH_Small" H 7650 4150 50  0001 C CNN
-F 3 "" H 7650 4150 50  0001 C CNN
-	1    7650 4150
+P 7650 4250
+F 0 "TP8" H 7650 4550 50  0000 C BNN
+F 1 "TEST" H 7650 4500 50  0000 C CNN
+F 2 "Measurement_Points:Measurement_Point_Round-TH_Small" H 7650 4250 50  0001 C CNN
+F 3 "" H 7650 4250 50  0001 C CNN
+	1    7650 4250
 	0    1    1    0
 $EndComp
@@
 L TEST TP9
 U 1 1 59FD805A
-P 7650 4900
-F 0 "TP9" H 7650 5200 50  0000 C BNN
-F 1 "TEST" H 7650 5150 50  0000 C CNN
-F 2 "Measurement_Points:Measurement_Point_Round-TH_Small" H 7650 4900 50  0001 C CNN
-F 3 "" H 7650 4900 50  0001 C CNN
-	1    7650 4900
+P 7650 4750
+F 0 "TP9" H 7650 5050 50  0000 C BNN
+F 1 "TEST" H 7650 5000 50  0000 C CNN
+F 2 "Measurement_Points:Measurement_Point_Round-TH_Small" H 7650 4750 50  0001 C CNN
+F 3 "" H 7650 4750 50  0001 C CNN
+	1    7650 4750
 	0    1    1    0
 $EndComp
@@
 P 2150 4700
 F 0 "R4" V 2230 4700 50  0000 C CNN
-F 1 "10k" V 2150 4700 50  0000 C CNN
+F 1 "12k" V 2150 4700 50  0000 C CNN
 F 2 "Resistors_SMD:R_0805_HandSoldering" V 2080 4700 50  0001 C CNN
 F 3 "" H 2150 4700 50  0001 C CNN
@@
 P 2150 5100
 F 0 "R5" V 2230 5100 50  0000 C CNN
-F 1 "5.6k" V 2150 5100 50  0000 C CNN
+F 1 "20k" V 2150 5100 50  0000 C CNN
 F 2 "Resistors_SMD:R_0805_HandSoldering" V 2080 5100 50  0001 C CNN
 F 3 "" H 2150 5100 50  0001 C CNN
@@
 	3600 5350 5050 5350
 Wire Wire Line
-	3600 5450 5050 5450
+	3450 5450 5050 5450
 Wire Wire Line
 	3600 5550 5050 5550
 Wire Wire Line
-	3600 5650 5050 5650
-Wire Wire Line
-	5250 6900 5250 7700
-Wire Wire Line
-	5250 7500 5500 7500
-Wire Wire Line
-	5250 7200 5500 7200
-Connection ~ 5250 7500
-Wire Wire Line
-	5250 6900 5500 6900
-Connection ~ 5250 7200
+	3500 5650 5050 5650
+Wire Wire Line
+	4850 6850 4850 7650
+Wire Wire Line
+	4850 7450 5100 7450
+Wire Wire Line
+	4850 7150 5100 7150
+Connection ~ 4850 7450
+Wire Wire Line
+	4850 6850 5100 6850
+Connection ~ 4850 7150
 Wire Wire Line
 	3300 3800 2850 3800
@@
 Wire Wire Line
 	4400 1600 4400 1800
+Wire Wire Line
+	3250 5500 3600 5500
+Wire Wire Line
+	3600 5500 3600 5550
+Wire Wire Line
+	3500 5650 3500 5550
+Wire Wire Line
+	3500 5550 3050 5550
+Wire Wire Line
+	3050 5550 3050 5500
+Wire Wire Line
+	7650 4900 7650 4750
+Wire Wire Line
+	7650 5100 7650 5000
+Wire Wire Line
+	7650 4150 7650 4250
 $EndSCHEMATC

Commit message: Working on rev 3, started board layout
Parts:
- removed C2: 10n, Capacitors_SMD:C_0805_HandSoldering, symbol C
- removed C8: DNI, Capacitors_SMD:C_0805_HandSoldering, symbol C
- removed D1: 5.6V Zener, tracking_device:DO-214AC, symbol D_Zener
- removed J2: CONN_COAXIAL, tracking_device:RP-SMA, symbol CONN_COAXIAL
- removed L1: 27n, Inductors_SMD:L_0805_HandSoldering, symbol L
- removed Q1: PMGD280UN, tracking_device:SOT-363_SC-70-6_Handsoldering, symbol PMGD280UN
- removed R1: 10, Resistors_SMD:R_0805_HandSoldering, symbol R
- removed R11, R13, R14, R2: 10k, Resistors_SMD:R_0805_HandSoldering, symbol R
- removed R12: 100, Resistors_SMD:R_0805_HandSoldering, symbol R
- removed R3, R5: 20k, Resistors_SMD:R_0805_HandSoldering, symbol R
- removed R4: 12k, Resistors_SMD:R_0805_HandSoldering, symbol R
- removed R6: DNI, Resistors_SMD:R_0805_HandSoldering, symbol R
- removed SW1, SW2: SW_SPDT, tracking_device:CSS-1210TB, symbol SW_SPDT
- removed TP6: TEST, Measurement_Points:Measurement_Point_Round-TH_Small, symbol TEST
- removed U2: LDK220M30R, tracking_device:SOT-23-5_HandSoldering, symbol LDK220
- removed U3: MAX-M8, tracking_device:U-BLOX_MAX-M8, symbol MAX-M8
- added D2: NSR0320MW2T1G, Diodes_SMD:D_SOD-323_HandSoldering, symbol D_Schottky
- added Q1: Si2343DS, TO_SOT_Packages_SMD:SOT-23_Handsoldering, symbol Q_PMOS_GSD
- added SW? (x2): PUSH, symbol PUSH
- added U2: SAM-M8, tracking_device:SAM-M8, symbol SAM-M8
- added U5: REG113NA-3.3, tracking_device:SOT-23-5_HandSoldering, symbol REG113
- C11: renamed from C1; value 1u -> 100n
- C12: renamed from C4; value 1u -> 4.7u
- J6: renamed from J7; footprint tracking_device:JST_PH_S2B-PH-SM4-TB_02x2.00mm_Angled -> tracking_device:PH-2AWD
- R16: value 12k -> 10k
- R6: renamed from R15; value 4k -> 12k
- renumbered C6 to C1, C14 to C10, C7 to C2, C5 to C4, C9 to C5, C10 to C6, C11 to C7, C12 to C8, C13 to C9, J3 to J2, J4 to J3, J5 to J4, J6 to J5, J8 to J7, R10 to R1, R18 to R10, R19 to R11, R20 to R12, R21 to R13, R22 to R14, R23 to R15, R7 to R2, R8 to R3, R9 to R4, R17 to R7, R24 to R8, R25 to R9, TP11 to TP10, TP5 to TP2, TP4 to TP3, TP3 to TP4, TP2 to TP5, TP7 to TP6, TP8 to TP7, TP9 to TP8, TP10 to TP9, U4 to U3, U5 to U4
Connections:
- net VUSB_DET is gone; now on net VUSB: TP5.1
- net GND: now also R6.1, SW?.2, SW?.2, U2.10 (GND), U2.11 (GND), U2.15 (GND), U2.16 (GND), U2.20 (GND), U2.4 (GND), U2.5 (GND), U2.6 (GND), U5.2 (GND)
- net GPS_EXTINT: now also U2.19 (EXTINT)
- net GPS_RESET_N: now also U2.18 (RESET_N)
- net GPS_TIMEPULSE: now also U2.7 (TIMEPULSE)
- net GPS_UART_RX: now also R2.1; no longer R3.1
- net GPS_UART_TX: now also R3.1; no longer R2.1
- net Microcontroller/SWITCH_1: now also SW?.1
- net Microcontroller/SWITCH_2: now also SW?.1
- net VBAT: now also Q1.3 (D); no longer C11.2
- net VDD: now also U2.1 (GND), U2.17 (VCC), U2.2 (VCC_IO), U2.3 (V_BCKP), U5.5 (OUT)
- net VUSB: now also R16.1, D2.2 (A), Q1.1 (G)
- net at R6.2, U3.5 (PROG): no longer R16.1
- net at R1.2: now also U2.9 (SDA)
- net at R4.2: now also U2.12 (SCL)
- net at R2.2: now also U2.14 (RXD)
- net at R3.2: now also U2.13 (TXD)
- new net: C11.2, D2.1 (K), Q1.2 (S), U5.1 (IN), U5.3 (EN)
- no-connect marks 5 -> 3
Other:
- note removed: "VCC_RF is for powering active\nantenna if it also operates at VCC\nDNI inductor if not used"
- moved on the sheet: C1, C11, C12, C2, C3, C4, C5, C6, C7, C8, J1, J5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
